Commit message: spawned

File: chipta_bot/urdf/chipta.xacro (robot description, xacro)
@@ -1,7 +1,7 @@
 <?xml version="1.0" ?>
 <robot name="chipta" xmlns:xacro="http://www.ros.org/wiki/xacro">
-<xacro:include filename="$(find chipta_description)/urdf/materials.xacro" />
-<xacro:include filename="$(find chipta_description)/urdf/chipta.ros2control" />
-<xacro:include filename="$(find chipta_description)/urdf/chipta.gazebo" />
+<xacro:include filename="$(find chipta_bot)/urdf/materials.xacro" />
+<xacro:include filename="$(find chipta_bot)/urdf/chipta.ros2control" />
+<xacro:include filename="$(find chipta_bot)/urdf/chipta.gazebo" />
 <link name="base_link">
   <inertial>
@@ -13,5 +13,5 @@
     <origin xyz="0 0 0" rpy="0 0 0"/>
     <geometry>
-      <mesh filename="file://$(find chipta_description)/meshes/base_link.stl" scale="0.001 0.001 0.001"/>
+      <mesh filename="file://$(find chipta_bot)/meshes/base_link.stl" scale="0.001 0.001 0.001"/>
     </geometry>
     <material name="silver"/>
@@ -20,5 +20,5 @@
     <origin xyz="0 0 0" rpy="0 0 0"/>
     <geometry>
-      <mesh filename="file://$(find chipta_description)/meshes/base_link.stl" scale="0.001 0.001 0.001"/>
+      <mesh filename="file://$(find chipta_bot)/meshes/base_link.stl" scale="0.001 0.001 0.001"/>
     </geometry>
   </collision>
@@ -33,5 +33,5 @@
     <origin xyz="-0.005 -0.0 -0.015" rpy="0 0 0"/>
     <geometry>
-      <mesh filename="file://$(find chipta_description)/meshes/IMU_v1_1.stl" scale="0.001 0.001 0.001"/>
+      <mesh filename="file://$(find chipta_bot)/meshes/IMU_v1_1.stl" scale="0.001 0.001 0.001"/>
     </geometry>
     <material name="silver"/>
@@ -40,5 +40,5 @@
     <origin xyz="-0.005 -0.0 -0.015" rpy="0 0 0"/>
     <geometry>
-      <mesh filename="file://$(find chipta_description)/meshes/IMU_v1_1.stl" scale="0.001 0.001 0.001"/>
+      <mesh filename="file://$(find chipta_bot)/meshes/IMU_v1_1.stl" scale="0.001 0.001 0.001"/>
     </geometry>
   </collision>
@@ -53,5 +53,5 @@
     <origin xyz="0.03 -0.0 -0.018" rpy="0 0 0"/>
     <geometry>
-      <mesh filename="file://$(find chipta_description)/meshes/GPS_v1_1.stl" scale="0.001 0.001 0.001"/>
+      <mesh filename="file://$(find chipta_bot)/meshes/GPS_v1_1.stl" scale="0.001 0.001 0.001"/>
     </geometry>
     <material name="silver"/>
@@ -60,5 +60,5 @@
     <origin xyz="0.03 -0.0 -0.018" rpy="0 0 0"/>
     <geometry>
-      <mesh filename="file://$(find chipta_description)/meshes/GPS_v1_1.stl" scale="0.001 0.001 0.001"/>
+      <mesh filename="file://$(find chipta_bot)/meshes/GPS_v1_1.stl" scale="0.001 0.001 0.001"/>
     </geometry>
   </collision>
@@ -73,5 +73,5 @@
     <origin xyz="-0.1125 0.0015 -0.04" rpy="0 0 0"/>
     <geometry>
-      <mesh filename="file://$(find chipta_description)/meshes/Lidar_v1_1.stl" scale="0.001 0.001 0.001"/>
+      <mesh filename="file://$(find chipta_bot)/meshes/Lidar_v1_1.stl" scale="0.001 0.001 0.001"/>
     </geometry>
     <material name="silver"/>
@@ -80,5 +80,5 @@
     <origin xyz="-0.1125 0.0015 -0.04" rpy="0 0 0"/>
     <geometry>
-      <mesh filename="file://$(find chipta_description)/meshes/Lidar_v1_1.stl" scale="0.001 0.001 0.001"/>
+      <mesh filename="file://$(find chipta_bot)/meshes/Lidar_v1_1.stl" scale="0.001 0.001 0.001"/>
     </geometry>
   </collision>
@@ -93,5 +93,5 @@
     <origin xyz="-0.064778 -0.085 -0.030131" rpy="0 0 0"/>
     <geometry>
-      <mesh filename="file://$(find chipta_description)/meshes/Wheel_front_left_1.stl" scale="0.001 0.001 0.001"/>
+      <mesh filename="file://$(find chipta_bot)/meshes/Wheel_front_left_1.stl" scale="0.001 0.001 0.001"/>
     </geometry>
     <material name="silver"/>
@@ -100,5 +100,5 @@
     <origin xyz="-0.064778 -0.085 -0.030131" rpy="0 0 0"/>
     <geometry>
-      <mesh filename="file://$(find chipta_description)/meshes/Wheel_front_left_1.stl" scale="0.001 0.001 0.001"/>
+      <mesh filename="file://$(find chipta_bot)/meshes/Wheel_front_left_1.stl" scale="0.001 0.001 0.001"/>
     </geometry>
   </collision>
@@ -113,5 +113,5 @@
     <origin xyz="-0.064778 0.085 -0.030131" rpy="0 0 0"/>
     <geometry>
-      <mesh filename="file://$(find chipta_description)/meshes/Wheel_front_right_1.stl" scale="0.001 0.001 0.001"/>
+      <mesh filename="file://$(find chipta_bot)/meshes/Wheel_front_right_1.stl" scale="0.001 0.001 0.001"/>
     </geometry>
     <material name="silver"/>
@@ -120,5 +120,5 @@
     <origin xyz="-0.064778 0.085 -0.030131" rpy="0 0 0"/>
     <geometry>
-      <mesh filename="file://$(find chipta_description)/meshes/Wheel_front_right_1.stl" scale="0.001 0.001 0.001"/>
+      <mesh filename="file://$(find chipta_bot)/meshes/Wheel_front_right_1.stl" scale="0.001 0.001 0.001"/>
     </geometry>
   </collision>
@@ -133,5 +133,5 @@
     <origin xyz="0.064941 0.085 -0.031781" rpy="0 0 0"/>
     <geometry>
-      <mesh filename="file://$(find chipta_description)/meshes/Wheel_rear_right_1.stl" scale="0.001 0.001 0.001"/>
+      <mesh filename="file://$(find chipta_bot)/meshes/Wheel_rear_right_1.stl" scale="0.001 0.001 0.001"/>
     </geometry>
     <material name="silver"/>
@@ -140,5 +140,5 @@
     <origin xyz="0.064941 0.085 -0.031781" rpy="0 0 0"/>
     <geometry>
-      <mesh filename="file://$(find chipta_description)/meshes/Wheel_rear_right_1.stl" scale="0.001 0.001 0.001"/>
+      <mesh filename="file://$(find chipta_bot)/meshes/Wheel_rear_right_1.stl" scale="0.001 0.001 0.001"/>
     </geometry>
   </collision>
@@ -153,5 +153,5 @@
     <origin xyz="0.064941 -0.085 -0.030131" rpy="0 0 0"/>
     <geometry>
-      <mesh filename="file://$(find chipta_description)/meshes/Wheel_rear_left_1.stl" scale="0.001 0.001 0.001"/>
+      <mesh filename="file://$(find chipta_bot)/meshes/Wheel_rear_left_1.stl" scale="0.001 0.001 0.001"/>
     </geometry>
     <material name="silver"/>
@@ -160,5 +160,5 @@
     <origin xyz="0.064941 -0.085 -0.030131" rpy="0 0 0"/>
     <geometry>
-      <mesh filename="file://$(find chipta_description)/meshes/Wheel_rear_left_1.stl" scale="0.001 0.001 0.001"/>
+      <mesh filename="file://$(find chipta_bot)/meshes/Wheel_rear_left_1.stl" scale="0.001 0.001 0.001"/>
     </geometry>
   </collision>

Commit message: files

File: chipta_bot/urdf/chipta.xacro (robot description, xacro)
@@ -15,5 +15,5 @@
       <mesh filename="file://$(find chipta_bot)/meshes/base_link.stl" scale="0.001 0.001 0.001"/>
     </geometry>
-    <material name="silver"/>
+    <material name="purple"/>
   </visual>
   <collision>
@@ -95,5 +95,5 @@
       <mesh filename="file://$(find chipta_bot)/meshes/Wheel_front_left_1.stl" scale="0.001 0.001 0.001"/>
     </geometry>
-    <material name="silver"/>
+    <material name="black"/>
   </visual>
   <collision>
@@ -115,5 +115,5 @@
       <mesh filename="file://$(find chipta_bot)/meshes/Wheel_front_right_1.stl" scale="0.001 0.001 0.001"/>
     </geometry>
-    <material name="silver"/>
+    <material name="black"/>
   </visual>
   <collision>
@@ -135,5 +135,5 @@
       <mesh filename="file://$(find chipta_bot)/meshes/Wheel_rear_right_1.stl" scale="0.001 0.001 0.001"/>
     </geometry>
-    <material name="silver"/>
+    <material name="black"/>
   </visual>
   <collision>
@@ -155,5 +155,5 @@
       <mesh filename="file://$(find chipta_bot)/meshes/Wheel_rear_left_1.stl" scale="0.001 0.001 0.001"/>
     </geometry>
-    <material name="silver"/>
+    <material name="black"/>
   </visual>
   <collision>

File: chipta_bot/urdf/materials.xacro (robot description, xacro)
@@ -4,3 +4,9 @@
   <color rgba="0.700 0.700 0.700 1.000"/>
 </material>
+<material name="purple">
+  <color rgba="0.5 0.0 0.7 1.0"/>
+</material>
+<material name="black">
+  <color rgba="0 0 0 1"/>
+</material>
 </robot>
