Commit message: mock component ros2_control

File: helios_description/urdf/helios_description.xacro (robot description, xacro)
@@ -2,6 +2,7 @@
 <robot name="chipta" xmlns:xacro="http://www.ros.org/wiki/xacro">
 <xacro:include filename="$(find helios_description)/urdf/materials.xacro" />
-<xacro:include filename="$(find helios_description)/urdf/helios_description.ros2control" />
+<xacro:include filename="$(find helios_description)/urdf/helios_description.ros2control.xacro" />
 <xacro:include filename="$(find helios_description)/urdf/helios_description.gazebo" />
+<link name="base_footprint"/>
 <link name="base_link">
   <inertial>
@@ -164,4 +165,9 @@
   </collision>
 </link>
+<joint name="fixed_base_joint" type="fixed">
+  <parent link="base_footprint" />
+  <child link="base_link" />
+  <origin xyz="0 0 0" rpy="0 0 0" />
+</joint>
 <joint name="Rigid 14" type="fixed">
   <origin xyz="0.005 0.0 0.015" rpy="0 0 0"/>
@@ -189,5 +195,5 @@
   <parent link="base_link"/>
   <child link="Wheel_front_right_1"/>
-  <axis xyz="0.0 -1.0 0.0"/>
+  <axis xyz="0.0 1.0 0.0"/>
 </joint>
 <joint name="wheel_rear_right_joint" type="continuous">
