Commit message: ros2_control gazebo wheels tf needs to be fixed

File: helios_description/urdf/helios_description.ros2control.xacro (robot description, xacro)
@@ -4,27 +4,28 @@
     <ros2_control name="HeliosBaseHardwareInterface" type="system">
         <hardware>
-            <plugin>mock_components/GenericSystem</plugin>
+            <!-- <plugin>mock_components/GenericSystem</plugin> -->
+            <plugin>gz_ros2_control/GazeboSimSystem</plugin>
             <param name="calculate_dynamics">true</param>
         </hardware>
-    <joint name="wheel_front_left_joint">
-        <command_interface name="velocity" />
-        <state_interface name="position" />
-        <state_interface name="velocity" />
-    </joint>
-    <joint name="wheel_front_right_joint">
-        <command_interface name="velocity" />
-        <state_interface name="position" />
-        <state_interface name="velocity" />
-    </joint>
-    <joint name="wheel_rear_right_joint">
-        <command_interface name="velocity" />
-        <state_interface name="position" />
-        <state_interface name="velocity" />
-    </joint>
-    <joint name="wheel_rear_left_joint">
-        <command_interface name="velocity" />
-        <state_interface name="position" />
-        <state_interface name="velocity" />
-    </joint>
+        <joint name="wheel_front_left_joint">
+            <command_interface name="velocity" />
+            <state_interface name="position" />
+            <state_interface name="velocity" />
+        </joint>
+        <joint name="wheel_front_right_joint">
+            <command_interface name="velocity" />
+            <state_interface name="position" />
+            <state_interface name="velocity" />
+        </joint>
+        <joint name="wheel_rear_right_joint">
+            <command_interface name="velocity" />
+            <state_interface name="position" />
+            <state_interface name="velocity" />
+        </joint>
+        <joint name="wheel_rear_left_joint">
+            <command_interface name="velocity" />
+            <state_interface name="position" />
+            <state_interface name="velocity" />
+        </joint>
     </ros2_control>
 </robot>
